File: HBridge84.sch (EAGLE design)
At the start: 21 parts, among them J5 ICSP

Commit message: adding eagle files
Parts:
- removed D1, D2, D3, D4, D5, D6, D7, D8: (no value), SparkFun-DiscreteSemi:DIODEPTH
- removed JP1, JP2, M1, M2: (no value), SparkFun-Connectors:M02PTH
- added C2: (no value), barbary_enterprises:CAPPTH
- added U$1, U$10, U$3, U$4, U$5, U$6, U$8, U$9: M1, barbary_enterprises:M1
- added U$7: RJ12, barbary_enterprises:RJ12
Connections:
- net 10: now also SN754410.IN2; no longer SN754410.IN1
- net 2: now also SN754410.IN3; no longer J2.3
- net 3: now also SN754410.IN4; no longer J3.3
- net 4: now also J2.3, U$7.4_GREEN; no longer J4.3
- net 5: now also J3.3, U$7.5_YELLOW; no longer SN754410.IN3
- net 5V: now also C2.1, U$10.P$1, U$7.3_RED; no longer JP1.2
- net 6: now also J4.3, U$7.6_BLUE; no longer SN754410.IN4
- net 7: now also SN754410.EN12; no longer SN754410.EN34
- net 8: now also SN754410.EN34; no longer SN754410.IN2
- net 9: now also SN754410.IN1; no longer SN754410.EN12
- net GND: now also C2.2, RESET.1, U$7.2_BLACK, U$8.P$1, U$9.P$1; no longer D2.A, D4.A, D6.A, D8.A, JP1.1, JP2.1
- net OUT1: now also U$1.P$1; no longer D1.A, D2.C, M1.2
- net OUT2: now also U$3.P$1; no longer D3.A, D4.C, M1.1
- net OUT3: now also U$4.P$1; no longer D5.A, D6.C, M2.1
- net OUT4: now also U$5.P$1; no longer D7.A, D8.C, M2.2
- net RST: now also RESET.4, U$7.1_WHITE
- net V_BATT: now also U$6.P$1; no longer D1.C, D3.C, D5.C, D7.C, JP2.2
Other:
- moved on the sheet: J5, RESET
