File: RJ11-ICSP-Breakout.sch (EAGLE design)
At the start: 3 parts, among them J5 ICSP

Commit message: updating ICSP breakout
Parts:
- removed JP1: (no value), SparkFun-Connectors:M06SILK_FEMALE_PTH
Connections:
- net 4: no longer JP1.4
- net 5: no longer JP1.5
- net 5V: no longer JP1.3
- net 6: no longer JP1.6
- net GND: no longer JP1.2
- net RST: no longer JP1.1
Changed lines of the file:
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@@
 <part name="GND13" library="SparkFun-Aesthetics" deviceset="GND" device=""/>
 <part name="U$7" library="barbary_enterprises" deviceset="RJ12" device=""/>
-<part name="JP1" library="SparkFun-Connectors" deviceset="M06" device="SILK_FEMALE_PTH"/>
 </parts>
 <sheets>
@@
 <instance part="GND13" gate="1" x="50.8" y="60.96"/>
 <instance part="U$7" gate="G$1" x="73.66" y="68.58" rot="R180"/>
-<instance part="JP1" gate="G$1" x="91.44" y="68.58" rot="MR0"/>
 </instances>
 <busses>
@@
 <wire x1="78.74" y1="66.04" x2="86.36" y2="66.04" width="0.1524" layer="91"/>
 <label x="81.28" y="66.04" size="1.778" layer="95"/>
-<pinref part="JP1" gate="G$1" pin="2"/>
 </segment>
 </net>
@@
 <wire x1="78.74" y1="68.58" x2="86.36" y2="68.58" width="0.1524" layer="91"/>
 <label x="81.28" y="68.58" size="1.778" layer="95"/>
-<pinref part="JP1" gate="G$1" pin="3"/>
 </segment>
 </net>
@@
 <pinref part="U$7" gate="G$1" pin="4_GREEN"/>
 <label x="81.28" y="71.12" size="1.778" layer="95"/>
-<pinref part="JP1" gate="G$1" pin="4"/>
 <wire x1="78.74" y1="71.12" x2="86.36" y2="71.12" width="0.1524" layer="91"/>
 </segment>
@@
 <pinref part="U$7" gate="G$1" pin="5_YELLOW"/>
 <label x="81.28" y="73.66" size="1.778" layer="95"/>
-<pinref part="JP1" gate="G$1" pin="5"/>
 <wire x1="78.74" y1="73.66" x2="86.36" y2="73.66" width="0.1524" layer="91"/>
 </segment>
@@
 <pinref part="U$7" gate="G$1" pin="6_BLUE"/>
 <label x="81.28" y="76.2" size="1.778" layer="95"/>
-<pinref part="JP1" gate="G$1" pin="6"/>
 <wire x1="78.74" y1="76.2" x2="86.36" y2="76.2" width="0.1524" layer="91"/>
 </segment>
@@
 <pinref part="U$7" gate="G$1" pin="1_WHITE"/>
 <label x="81.28" y="63.5" size="1.778" layer="95"/>
-<pinref part="JP1" gate="G$1" pin="1"/>
 <wire x1="78.74" y1="63.5" x2="86.36" y2="63.5" width="0.1524" layer="91"/>
 </segment>
